File: initial/z80computer/z80computer/z80computer.kicad_pcb (KiCad board)
At the start: 2 copper layers, 122.8 x 113.3 mm, 11 parts, among them J1 Conn_02x20_Top_Bottom, J2 Conn_02x03_Top_Bottom, U4 Z80CPU

Commit message: added kicad template for board designs. also has currentv version of the boards ( back plane and processor board)
Parts:
- J1: value Conn_02x20_Top_Bottom -> pin header 855-M20-9953645
Connections:
- net /VCC renamed /VCC5
- net Net-(J2-Pad4) renamed /VCC3

Commit message: version 1 circuit boards
Other:
- board size 122.8 x 113.3 mm -> 122.4 x 113.3 mm
