File: initial/z80computer/z80logic/z80logic.sch (KiCad schematic (older format))
At the start: 4 parts, among them J1 pin header 855-M20-9953645, J2 Conn_02x03_Top_Bottom

Commit message: version 1 circuit boards
Parts:
- added ANDWAIT1: SN74HC21N, Package_DIP:DIP-14_W7.62mm_Socket, symbol circuit_boards:SN74HC21N
- added C10, C11, C6: perf_12x4symbol, circuit_boards:perf_12x4, symbol circuit_boards:perf_12x4symbol
- added C12, C13, C2, C4: perf_9x4symbol, circuit_boards:perf_9x4, symbol circuit_boards:perf_9x4symbol
- added C14, C15, C16, C17, C18, C19, C20, C5: perf_13x4symbol, circuit_boards:perf_13x4, symbol circuit_boards:perf_13x4symbol
- added C7, C8: perf_36x4symbol, circuit_boards:perf_36x4, symbol circuit_boards:perf_36x4symbol
- added C9: 0.1uF, Capacitor_THT:C_Axial_L5.1mm_D3.1mm_P7.50mm_Horizontal, symbol Device:C_Small
- added CLOCK1: PIC18F24Q10-xSP, Package_DIP:DIP-28_W7.62mm, symbol circuit_boards:PIC18F24Q10-xSP
- added IOPORT1: GAL16V8, Package_DIP:DIP-20_W7.62mm_Socket, symbol circuit_boards:GAL16V8
- added J3: Conn_02x03_Odd_Even, Connector_PinSocket_2.54mm:PinSocket_2x03_P2.54mm_Vertical, symbol Connector_Generic:Conn_02x03_Top_Bottom
- added MEMCHIPSELECT1: MEMCHIPSELECT, Package_DIP:DIP-20_W7.62mm_Socket, symbol circuit_boards:GAL16V8
- added OR1: SN74LS32N, Package_DIP:DIP-14_W7.62mm_Socket, symbol circuit_boards:SN74LS32N
- added R1, R2: 1K, Resistor_THT:R_Axial_DIN0207_L6.3mm_D2.5mm_P10.16mm_Horizontal, symbol Device:R_Small_US
- added SW1: SW_SPST, Button_Switch_THT:SW_PUSH_6mm_H8mm, symbol Switch:SW_SPST
Connections:
- net labels added: 17, 18, 27, 28, 42, 43, 44, 48, 49, 50, 54, 55, 56, 60, 61, 62, 63, 64, 65, 66, 67, 68, 69, 70, 71, 72, A1A, A1B, A1C, A1D, A1Y, A2A, A2B, A2C, A2D, A2Y, O1A, O1B, O1Y, O2A, O2B, O2Y, O3A, O3B, O3Y, O4A, O4B, O4Y, POWER2, POWER3, PUSH
- wire segments 57 -> 845
Other:
- moved on the sheet: C1, C3, J1, J2
